File: stm32_nrf24/stm32_nrf24.kicad_pcb (KiCad board)
At the start: 2 copper layers, 74.4 x 30.3 mm, 54 parts, among them J1 USB_B_Micro, J2 Conn_01x03_Male, J3 Conn_Coaxial, J4 Conn_01x10_Male, J5 Conn_01x04_Female, SW1 SW_Push, U1 USBLC6-2SC6, U2 AMS1117-3.3, U3 STM32F103C8Tx, U4 RFX2401C, U5 nRF24L01P, Y1 Crystal_GND24, Y2 Crystal_GND24

Commit message: a
Parts:
- added G***: LOGO, stm32_nrf24:pusheen1, F.Cu at (139.9, 118.2)
Routing:
- net USB_D+: track 15.6 -> 16.3 mm
- net GND: vias 260 -> 259
- net +5V: vias 1 -> 0
