File: stm32_nrf24/stm32_stepper/stm32_stepper/stm32_stepper.kicad_pcb (KiCad board)
At the start: 2 copper layers, 83.6 x 102.6 mm, 53 parts, among them J1 USB_B_Micro, J10 Conn_01x04_Male, J11 Conn_01x02_Male, J12 Conn_01x02_Male, J13 Conn_01x02_Male, J14 Conn_01x04_Male, J15 Conn_01x02_Male, J16 Conn_01x02_Male, J17 Conn_01x02_Male, J18 Conn_01x03_Male, J19 Conn_01x04_Male, J2 Conn_01x02_Male, J3 Conn_01x02_Male, J4 Conn_01x02_Male, J5 Conn_01x04_Male, J6 Screw_Terminal_01x02, J7 Conn_01x02_Male, J8 Conn_01x02_Male, J9 Conn_01x02_Male, U1 STM32F405RGTx, U2 LM2596S-5, U3 AMS1117-3.3, Y1 Crystal

Commit message: b
Parts:
- moved C5 54.9 mm to (147.3, 98.6)
- moved C9 54.0 mm to (120.9, 90.7)
- moved C3 51.7 mm to (143.8, 113.5)
- moved C14 42.0 mm to (149.0, 108.7)
- moved C10 42.0 mm to (126.5, 133.2)
- moved C1 42.0 mm to (122.5, 133.2)
- moved C12 42.0 mm to (138.5, 106.6)
- moved C13 42.0 mm to (134.4, 131.9)
- moved C16 42.0 mm to (143.6, 119.3)
- moved C17 42.0 mm to (145.0, 108.7)
- moved C4 42.0 mm to (142.4, 122.7)
- moved C6 42.0 mm to (134.4, 127.6)
- moved C7 42.0 mm to (149.3, 113.8)
- moved C8 42.0 mm to (149.3, 111.2)
- moved Y1 32.4 mm to (123.7, 115.1), turned to 90 degrees
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Routing:
- net +12V: track 111.3 -> 143.3 mm
- net Net-(A2-Pad6): track 0.00 -> 9.84 mm
- net Net-(A2-Pad3): track 0.00 -> 9.80 mm
- net Net-(A2-Pad5): track 0.00 -> 9.44 mm
- net Net-(A2-Pad4): track 0.00 -> 9.40 mm
- net Net-(A3-Pad3): track 0.00 -> 9.30 mm
- net Net-(A1-Pad3): track 0.00 -> 9.21 mm
- net Net-(A1-Pad6): track 0.00 -> 9.20 mm
- net Net-(A3-Pad6): track 0.00 -> 9.07 mm
- net Net-(A3-Pad4): track 0.00 -> 8.90 mm
- net Net-(A1-Pad4): track 0.00 -> 8.82 mm
- net Net-(A1-Pad5): track 0.00 -> 8.80 mm
- net Net-(A3-Pad5): track 0.00 -> 8.67 mm
- net GND: track 100.3 -> 98.2 mm
